File: H360/H360.kicad_pcb (KiCad board)
At the start: 2 copper layers, 164 parts, among them J1 TYPE-C-31-M-12, J2 S2B-PH-SM4-TB, Q1 2N7002, SW1 PWR, SW2 TS-1187-A-B-A-B, SW3 TS-1187-A-B-A-B, U1 SRV05-4-P-T7, U3 nRF52840_holyiot_18010, U4 XC6206P332MR-G, U5 BQ24075RGT

Commit message: first final
Parts:
- removed C1, C2: 100nF, Capacitor_SMD:C_0402_1005Metric
- removed D1: BSD3C051V, Diode_SMD:D_SOD-323
- removed L2: BLM15PX121N1D, Inductor_SMD:L_0402_1005Metric
- removed TP1, TP4: TestPoint, TestPoint:TestPoint_Pad_D1.0mm
- added REF**: PinHeader_1x05_P2.54mm_Vertical, Connector_PinHeader_2.54mm:PinHeader_1x05_P2.54mm_Vertical, F.Cu at (206.5, 162.0)
- BOOT: renamed from SW3; moved to B.Cu
- C3, C4, C5, C6, C7, C8, F1, J1, J2, Q1, R1, R10, R2, R3, R4, R5, R6, R7, R8, R9, SW1, U1, U3, U4, U5: moved to B.Cu
- L1: value BLM15PX121N1D -> BLM15PX121SN1D; moved to B.Cu
- RST: renamed from SW2; moved to B.Cu
- moved J2 337.1 mm to (78.0, 157.0), turned to -90 degrees
- moved R9 331.8 mm to (80.0, 142.0), turned to 90 degrees
- moved C4 331.4 mm to (72.5, 136.5), turned to 180 degrees
- moved Q1 330.4 mm to (77.5, 143.1), turned to 90 degrees
- moved R10 330.0 mm to (81.0, 142.0), turned to -90 degrees
- moved C3 328.2 mm to (75.0, 133.5), turned to -90 degrees
- moved R8 324.2 mm to (74.0, 137.0), turned to -90 degrees
- moved SW1 323.3 mm to (70.6, 142.1), turned to 90 degrees
- moved C5 321.9 mm to (81.0, 135.0), turned to -90 degrees
- moved R3 302.2 mm to (77.0, 139.5), turned to -90 degrees
- moved R6 299.5 mm to (78.5, 139.5), turned to -90 degrees
- moved U5 298.5 mm to (77.8, 135.8)
- moved R7 297.9 mm to (75.0, 137.0), turned to -90 degrees
- moved R4 297.4 mm to (81.0, 137.0), turned to -90 degrees
- moved U1 199.2 mm to (88.2, 111.0)
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Connections:
- F1 pad 2: Net-(C1-Pad2) -> +5V
- J1 pad A1_B12: <NO NET> -> GND
- J1 pad B1_A12: <NO NET> -> GND
- J1 pad S1: <NO NET> -> GND
- J1 pad S2: <NO NET> -> GND
- J1 pad S3: <NO NET> -> GND
- J1 pad S4: <NO NET> -> GND
- MX64 pad 1: COL13 -> COL12
- R1 pad 1: GNDPWR -> GND
- R2 pad 2: GNDPWR -> GND
- U3 pad 10: COL1 -> ROW3
- U3 pad 11: COL0 -> ROW2
- U3 pad 12: unconnected-(U3-P0.04-A-Pad12) -> ROW1
- U3 pad 13: unconnected-(U3-P0.05-A-Pad13) -> COL0
- U3 pad 15: ROW0 -> unconnected-(U3-P0.07-Pad15)
- U3 pad 16: ROW1 -> unconnected-(U3-P1.09-Pad16)
- U3 pad 17: ROW2 -> unconnected-(U3-P0.12-Pad17)
- U3 pad 18: ROW3 -> unconnected-(U3-P0.23-Pad18)
- U3 pad 19: ROW4 -> unconnected-(U3-P0.21-Pad19)
- U3 pad 2: COL9 -> COL14
- U3 pad 26: COL14 -> COL5
- U3 pad 27: COL13 -> COL6
- U3 pad 28: COL12 -> COL7
- U3 pad 29: COL11 -> COL9
- U3 pad 3: COL8 -> ROW4
- U3 pad 33: unconnected-(U3-P1.04-LF-Pad33) -> COL11
- U3 pad 34: unconnected-(U3-P1.06-LF-Pad34) -> COL12
- U3 pad 35: unconnected-(U3-P0.09-LF-NFC-Pad35) -> COL13
- U3 pad 36: unconnected-(U3-P0.10-LF-NFC-Pad36) -> COL8
- U3 pad 4: COL7 -> unconnected-(U3-P1.13-LF-Pad4)
- U3 pad 5: COL6 -> COL1
- U3 pad 6: COL5 -> COL2
- U3 pad 7: COL4 -> COL3
- U3 pad 8: COL3 -> COL4
- U3 pad 9: COL2 -> ROW0
Routing:
- net GND: track 0.00 -> 690.6 mm, vias 0 -> 18
- net ROW0: track 266.7 -> 502.2 mm, vias 0 -> 4
- net +5V: track 0.00 -> 213.0 mm, vias 0 -> 6
- net +VSW: track 0.00 -> 197.0 mm, vias 0 -> 2
- net D-: track 0.00 -> 194.4 mm
- net D+: track 0.00 -> 192.9 mm
- net ROW1: track 257.2 -> 445.9 mm, vias 0 -> 2
- net ROW2: track 247.6 -> 415.1 mm, vias 0 -> 2
- net COL12: track 44.1 -> 201.6 mm, vias 4 -> 1
- net ROW3: track 264.3 -> 413.2 mm, vias 0 -> 4
- net COL0: track 62.1 -> 207.8 mm, vias 0 -> 7
- net COL1: track 83.1 -> 219.5 mm, vias 8 -> 3
- net COL14: track 92.5 -> 215.8 mm, vias 8 -> 1
- net COL13: track 84.2 -> 203.3 mm, vias 8 -> 1
- net COL2: track 94.7 -> 202.5 mm, vias 8 -> 1
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Other:
- board outline added: 285 x 96.5 mm
- board text added: "3V3"
- board text added: "GND"
- board text added: "RST"
- board text added: "SWDCLK"
- board text added: "SWDIO"
