File: H360/H360.kicad_pcb (KiCad board)
At the start: 2 copper layers, 285 x 96.5 mm, 159 parts, among them J1 TYPE-C-31-M-12, J2 S2B-PH-SM4-TB, Q1 2N7002, SW1 PWR, U1 SRV05-4-P-T7, U3 nRF52840_holyiot_18010, U4 XC6206P332MR-G, U5 BQ24075RGT

Commit message: fixes
Parts:
- moved SW1 0.42 mm to (70.6, 142.5)
Routing:
- net COL5: track 127.8 -> 125.4 mm
- net GND: track 690.6 -> 691.9 mm, vias 18 -> 19
- net COL12: track 201.6 -> 202.6 mm
- net COL14: track 215.8 -> 216.6 mm
- net COL11: track 185.3 -> 186.0 mm
- net COL6: track 90.6 -> 91.2 mm
- net COL2: track 202.5 -> 203.0 mm
- net COL7: track 82.6 -> 83.1 mm

Commit message: fixed routing
Parts:
- moved SW1 0.14 mm to (70.5, 142.5)
Routing:
- net GND: track 691.9 -> 695.9 mm
- net COL13: track 203.3 -> 205.6 mm
- net +3.3V: track 43.9 -> 43.3 mm

Commit message: routing fixed
Routing:
- net GND: track 695.9 -> 701.1 mm
- net COL3: track 172.7 -> 173.4 mm

Commit message: else
Parts:
- C3, C4, C5: footprint Capacitor_SMD:C_0402_1005Metric -> Capacitor_SMD:C_0603_1608Metric
- C6, C7: footprint Capacitor_SMD:C_1812_4532Metric -> Capacitor_SMD:C_1206_3216Metric
- R3: footprint Resistor_SMD:R_0402_1005Metric -> Resistor_SMD:R_0603_1608Metric
- moved D32 2.79 mm to (90.5, 152.5), turned to 180 degrees
- moved C6 1.67 mm to (198.5, 187.7)
- moved C7 0.72 mm to (201.0, 187.7)
- moved C3 0.50 mm to (74.5, 133.5)
- moved C4 0.50 mm to (72.0, 136.5)
- moved C5 0.28 mm to (81.0, 134.7)
- moved R3 0.25 mm to (76.8, 139.5)
- moved R4 0.25 mm to (81.0, 137.2)
- renumbered RST to SW2, BOOT to SW3
Routing:
- net ROW2: track 415.1 -> 417.3 mm
- net GND: track 701.1 -> 703.1 mm, vias 19 -> 21
- net SYSOFF: track 10.6 -> 9.46 mm
- net +VSW: track 196.9 -> 196.1 mm
- net Net-(D32-A): track 9.40 -> 8.79 mm
- added copper zone on F.Cu, net GND

Commit message: 05.16
Routing:
- net ROW0: track 502.5 -> 501.7 mm
