File: H360/H360.kicad_sch (KiCad schematic)
At the start: 1 part, among them U1 TP4056-42-ESOP8

Commit message: sch updat4e
Parts:
- added C1, C2: 100nF, symbol Device:C_Small
- added C3: 4.7u, symbol Device:C_Small
- added C4, C5: 10u, symbol Device:C_Small
- added C6, C7: 1u, symbol Device:C_Small
- added C8: 100n, symbol Device:C_Small
- added D1: BSD3C051V, symbol Device:D_Small
- added D2: Schottky, symbol Device:D_Schottky
- added F1: MF-MSMF075-2, symbol Device:Fuse_Small
- added J1: TYPE-C-31-M-12, TYPE-C-31-M-12:HRO_TYPE-C-31-M-12, symbol TYPE-C-31-M-12:TYPE-C-31-M-12
- added J2: JST-PH 2.0, symbol Connector:Conn_01x02_Pin
- added L1, L2: BLM15PX121N1D, symbol Device:L_Small
- added Q1: AO3401A, Package_TO_SOT_SMD:SOT-23, symbol Transistor_FET:AO3401A
- added R1, R2: 5.1k, symbol Device:R_Small
- added R3: 5k, symbol Device:R_Small
- added R4: 1.5k, symbol Device:R_Small
- added SW1: SW_SPST, symbol Switch:SW_SPST
- added SW2: TS-1187A-B-A-B, symbol Switch:SW_MEC_5G
- added TP1, TP2, TP3: TestPoint, symbol Connector:TestPoint
- added U1: SRV05-4-P-T7, Package_TO_SOT_SMD:SOT-23-6, symbol Power_Protection:SRV05-4
- added U3: nRF52840_holyiot_18010, PCM_marbastlib-various:nRF52840_holyiot_18010, symbol base:nRF52840_holyiot_18010
- added U4: XC6206PxxxMR, Package_TO_SOT_SMD:SOT-23-3, symbol Regulator_Linear:XC6206PxxxMR
- renumbered U1 to U2
Connections:
- net GND: now reaches U2.1 (TEMP)
- net GND: now also U2.3 (GND), C2.2, C3.2, C4.2, C5.2, C6.2, C7.2, C8.2, D1.1 (K), J2.2 (Pin_2), L2.1, R3.2, R4.2, SW2.3 (B), SW2.4 (B), U1.2 (VN), U3.1 (GND), U3.25 (GND), U3.37 (GND), U4.1 (GND)
- net at U2.2 (PROG): now also R3.1
- net +5V: now reaches U2.4 (V_{CC})
- net +5V: now also U2.8 (CE), C1.1, C3.1, C4.1, D2.2 (A), Q1.1 (G), R4.1, U1.5 (VP), U3.22 (VBUS)
- net +BATT: now reaches U2.5 (BAT)
- net +BATT: now also C5.1, J2.1 (Pin_1), Q1.3 (D), TP2.1
- new net: J1.A4_B9 (VBUS), J1.B4_A9 (VBUS), L1.1, TP1.1
- new net: J1.B5 (CC2), R1.2
- new net: C2.1, D1.2 (A), J1.A1_B12 (GND), J1.B1_A12 (GND), J1.S1 (SHIELD), J1.S2 (SHIELD), J1.S3 (SHIELD), J1.S4 (SHIELD), L2.2
- new net: Q1.2 (S), SW1.1 (A)
- new net: J1.A5 (CC1), R2.1
- new net: F1.1, L1.2
- new net: C1.2, F1.2
- new net +3.3V: C7.1, C8.1, U3.14 (VDD_nRF), U4.2 (VO)
- new net +VSW: C6.1, D2.1 (K), SW1.2 (B), TP3.1, U4.3 (VI)
- new net D+: J1.A6 (DP1), J1.B6 (DP2), U1.6 (IO4), U3.24 (D+)
- new net D-: J1.A7 (DN1), J1.B7 (DN2), U1.1 (IO1), U3.23 (D-)
- new net GNDPWR: R1.1, R2.2
- new net RST: SW2.1 (A), SW2.2 (A), U3.21 (P0.18-RESET)
- no-connect marks 0 -> 6

Commit message: sch update
Parts:
- removed SW2: TS-1187A-B-A-B, symbol Switch:SW_MEC_5G
- added D10, D11, D12, D13, D14, D15, D16, D17, D18, D19, D20, D21, D22, D23, D24, D25, D26, D27, D28, D29, D3, D30, D31, D32, D33, D34, D35, D36, D37, D38, D39, D4, D40, D41, D42, D43, D44, D45, D46, D47, D48, D49, D5, D50, D51, D52, D53, D54, D55, D56, D57, D58, D59, D6, D60, D61, D62, D63, D64, D65, D66, D67, D7, D8, D9: D_Small, symbol Device:D_Small
- added MX1, MX10, MX11, MX12, MX13, MX14, MX15, MX16, MX17, MX18, MX19, MX2, MX20, MX21, MX22, MX23, MX24, MX25, MX26, MX27, MX28, MX29, MX3, MX30, MX31, MX32, MX33, MX34, MX35, MX36, MX37, MX38, MX39, MX4, MX40, MX41, MX42, MX43, MX44, MX45, MX46, MX47, MX48, MX49, MX5, MX50, MX51, MX52, MX53, MX54, MX55, MX56, MX57, MX58, MX59, MX6, MX60, MX61, MX62, MX63, MX64, MX65, MX7, MX8, MX9: MX_SW_HS, PCM_marbastlib-mx:SW_MX_HS_CPG151101S11_1u, symbol marbastlib-mx:MX_SW_HS_CPG151101S11
- added R5: 10k, symbol Device:R_Small
- added SW2, SW3: T-1187-A-B-A-B, symbol Switch:SW_Push
- added TP4: TestPoint, symbol Connector:TestPoint
Connections:
- net +3.3V: now also R5.1, TP4.1
- net GND: now also SW2.2, SW3.2
- net RST: now also SW2.1
- net COL1: now reaches U3.10 (P0.30-LF-A)
- net COL1: now also MX2.1, MX44.1, MX57.1
- net COL0: now reaches U3.11 (P0.31-LF-A)
- net COL0: now also MX1.1, MX16.1, MX30.1, MX43.1
- net ROW0: now reaches U3.15 (P0.07)
- net ROW0: now also D10.1 (K), D11.1 (K), D12.1 (K), D13.1 (K), D14.1 (K), D15.1 (K), D16.1 (K), D17.1 (K), D3.1 (K), D4.1 (K), D5.1 (K), D6.1 (K), D7.1 (K), D8.1 (K), D9.1 (K)
- net ROW1: now reaches U3.16 (P1.09)
- net ROW1: now also D18.1 (K), D19.1 (K), D20.1 (K)
- net ROW2: now reaches U3.17 (P0.12)
- net ROW2: now also D32.1 (K), D33.1 (K), D34.1 (K), D35.1 (K), D36.1 (K), D37.1 (K), D38.1 (K), D39.1 (K), D40.1 (K), D41.1 (K), D42.1 (K), D43.1 (K), D44.1 (K)
- net ROW3: now reaches U3.18 (P0.23)
- net ROW3: now also D45.1 (K), D46.1 (K), D47.1 (K), D48.1 (K), D49.1 (K), D50.1 (K), D51.1 (K), D52.1 (K), D53.1 (K), D54.1 (K), D55.1 (K), D56.1 (K), D57.1 (K), D58.1 (K)
- net ROW4: now reaches U3.19 (P0.21)
- net ROW4: now also D59.1 (K), D60.1 (K), D61.1 (K), D62.1 (K), D63.1 (K), D64.1 (K), D65.1 (K), D66.1 (K), D67.1 (K)
- net COL9: now reaches U3.2 (P1.11-LF)
- net COL9: now also MX10.1, MX24.1, MX38.1, MX52.1
- net BOOT: now reaches U3.20 (P0.19)
- net BOOT: now also R5.2, SW3.1
- net COL14: now reaches U3.26 (P0.22)
- net COL14: now also MX15.1, MX29.1, MX55.1
- net COL13: now reaches U3.27 (P1.00)
- net COL13: now also MX14.1, MX28.1, MX42.1, MX56.1, MX65.1
- net COL12: now reaches U3.28 (P1.03-LF)
- net COL12: now also MX13.1, MX27.1, MX41.1, MX64.1
- net COL11: now reaches U3.29 (P1.01-LF)
- net COL11: now also MX12.1, MX26.1, MX40.1, MX54.1, MX62.1
- net COL8: now reaches U3.3 (P1.10-LF)
- net COL8: now also MX23.1, MX37.1, MX51.1, MX61.1, MX9.1
- net COL10: now reaches U3.30 (P1.02-LF)
- net COL10: now also MX11.1, MX25.1, MX39.1, MX53.1, MX63.1
- net SWDCLK: now reaches U3.31 (SWDCLK)
- net SWDIO: now reaches U3.32 (SWDIO)
- net COL7: now reaches U3.4 (P1.13-LF)
- net COL7: now also MX22.1, MX36.1, MX50.1, MX8.1
- net COL6: now reaches U3.5 (P1.15-LF)
- net COL6: now also MX21.1, MX35.1, MX49.1, MX7.1
- net COL5: now reaches U3.6 (P0.03-LF-A)
- net COL5: now also MX20.1, MX34.1, MX48.1, MX6.1, MX60.1
- net COL4: now reaches U3.7 (P0.02-LF-A)
- net COL4: now also MX19.1, MX33.1, MX47.1, MX5.1
- net COL3: now reaches U3.8 (P0.28-LF-A)
- net COL3: now also MX18.1, MX32.1, MX4.1, MX46.1, MX59.1
- net COL2: now reaches U3.9 (P0.29-LF-A)
- net COL2: now also MX17.1, MX3.1, MX31.1, MX45.1, MX58.1
- new net: D58.2 (A), MX56.2
- new net: D49.2 (A), MX47.2
- new net: D31.2 (A), MX29.2
- new net: D33.2 (A), MX31.2
- new net: D8.2 (A), MX6.2
- new net: D59.2 (A), MX57.2
- new net: D34.2 (A), MX32.2
- new net: D67.2 (A), MX65.2
- new net: D42.2 (A), MX40.2
- new net: D17.2 (A), MX15.2
- new net: D43.2 (A), MX41.2
- new net: D7.2 (A), MX5.2
- new net: D56.2 (A), MX54.2
- new net: D61.2 (A), MX59.2
- new net: D64.2 (A), MX62.2
- new net: D24.1 (K), D25.1 (K), D26.1 (K), D27.1 (K), D28.1 (K), D29.1 (K), D30.1 (K), D31.1 (K)
- new net: D26.2 (A), MX24.2
- new net: D65.2 (A), MX63.2
- new net: D32.2 (A), MX30.2
- new net: D66.2 (A), MX64.2
- new net: D27.2 (A), MX25.2
- new net: D60.2 (A), MX58.2
- new net: D40.2 (A), MX38.2
- new net: D63.2 (A), MX61.2
- new net: D28.2 (A), MX26.2
- new net: D4.2 (A), MX2.2
- new net: D6.2 (A), MX4.2
- new net: D19.2 (A), MX17.2
- new net: D30.2 (A), MX28.2
- new net: D9.2 (A), MX7.2
- new net: D21.1 (K), D22.1 (K), D23.1 (K)
- new net: D21.2 (A), MX19.2
- new net: D20.2 (A), MX18.2
- new net: D36.2 (A), MX34.2
- new net: D48.2 (A), MX46.2
- new net: D12.2 (A), MX10.2
- new net: D51.2 (A), MX49.2
- new net: D52.2 (A), MX50.2
- new net: D23.2 (A), MX21.2
- new net: D37.2 (A), MX35.2
- new net: D45.2 (A), MX43.2
- new net: D44.2 (A), MX42.2
- new net: D54.2 (A), MX52.2
- new net: D22.2 (A), MX20.2
- new net: D3.2 (A), MX1.2
- new net: D57.2 (A), MX55.2
- new net: D10.2 (A), MX8.2
- new net: D62.2 (A), MX60.2
- new net: D18.2 (A), MX16.2
- new net: D5.2 (A), MX3.2
- new net: D35.2 (A), MX33.2
- new net: D41.2 (A), MX39.2
- new net: D55.2 (A), MX53.2
- new net: D25.2 (A), MX23.2
- new net: D14.2 (A), MX12.2
- new net: D13.2 (A), MX11.2
- new net: D39.2 (A), MX37.2
- new net: D53.2 (A), MX51.2
- new net: D46.2 (A), MX44.2
- new net: D16.2 (A), MX14.2
- new net: D47.2 (A), MX45.2
- new net: D24.2 (A), MX22.2
- new net: D11.2 (A), MX9.2
- new net: D50.2 (A), MX48.2
- new net: D29.2 (A), MX27.2
- new net: D38.2 (A), MX36.2
- new net: D15.2 (A), MX13.2
- no-connect marks 6 -> 29
Other:
- moved on the sheet: C1, C2, C3, C4, C5, C6, C7, C8, D1, D2, F1, J1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

Commit message: charger update
Parts:
- removed D2: Schottky, symbol Device:D_Schottky
- removed SW1: SW_SPST, symbol Switch:SW_SPST
- removed TP2, TP3: TestPoint, symbol Connector:TestPoint
- removed U2: TP4056-42-ESOP8, Package_SO:SOIC-8-1EP_3.9x4.9mm_P1.27mm_EP2.41x3.3mm_ThermalVias, symbol Battery_Management:TP4056-42-ESOP8
- added R10: 100R, symbol Device:R_Small
- added R6: 47k, symbol Device:R_Small
- added R7, R8, R9: 10k, symbol Device:R_Small
- added SW1: PWR, symbol Switch:SW_Push_SPDT
- added U5: BQ24075RGT, Package_DFN_QFN:VQFN-16-1EP_3x3mm_P0.5mm_EP1.6x1.6mm, symbol Battery_Management:BQ24075RGT
- C4, C5: value 10u -> 4.7u
- R3: value 5k -> 3.4k
Connections:
- net +5V: now also R10.1, U5.13 (IN); no longer C4.1, Q1.1 (G), R4.1
- net +BATT: now also C4.1, R8.1, U5.2 (BAT), U5.3 (BAT); no longer C5.1, Q1.3 (D)
- net +VSW: now also C5.1, U5.10 (OUT), U5.11 (OUT), U5.6 (EN1)
- net GND: now also Q1.2 (S), R6.2, R7.2, R9.2, SW1.3 (C), U5.17 (VSS), U5.4 (~{CE}), U5.5 (EN2), U5.8 (VSS)
- net at R3.1: now also U5.16 (ISET)
- new net: R8.2, SW1.1 (A)
- new net: R4.1, U5.12 (ILIM)
- new net: Q1.1 (G), R10.2, R9.1
- new net: R6.1, U5.14 (TMR)
- new net: R7.1, U5.1 (TS)
- new net SYSOFF: Q1.3 (D), SW1.2 (B), U5.15 (SYSOFF)
Other:
- moved on the sheet: J2, Q1

Commit message: ut
Parts:
- C1, C2, C3, C4, C5, C8: footprint (none) -> Capacitor_SMD:C_0402_1005Metric
- C6, C7: footprint (none) -> Capacitor_SMD:C_1812_4532Metric
- D1: footprint (none) -> Diode_SMD:D_SOD-323
- D10, D11, D12, D13, D14, D15, D16, D17, D18, D19, D20, D21, D22, D23, D24, D25, D26, D27, D28, D29, D3, D30, D31, D32, D33, D34, D35, D36, D37, D38, D39, D4, D40, D41, D42, D43, D44, D45, D46, D47, D48, D49, D5, D50, D51, D52, D53, D54, D55, D56, D57, D58, D59, D6, D60, D61, D62, D63, D64, D65, D66, D67, D7, D8, D9: footprint (none) -> Diode_SMD:D_SOD-123
- F1: footprint (none) -> Resistor_SMD:R_1812_4532Metric
- J1: footprint TYPE-C-31-M-12:HRO_TYPE-C-31-M-12 -> typeC:HRO_TYPE-C-31-M-12
- J2: value JST-PH 2.0 -> S2B-PH-SM4-TB; footprint (none) -> Connector_JST:JST_PH_S2B-PH-SM4-TB_1x02-1MP_P2.00mm_Horizontal
- L1, L2: footprint (none) -> Inductor_SMD:L_0402_1005Metric
- MX1, MX10, MX11, MX12, MX13, MX14, MX15, MX16, MX17, MX18, MX19, MX2, MX20, MX21, MX22, MX23, MX24, MX25, MX26, MX27, MX28, MX29, MX3, MX30, MX31, MX32, MX33, MX34, MX35, MX36, MX37, MX38, MX39, MX4, MX40, MX41, MX42, MX43, MX44, MX45, MX46, MX47, MX48, MX49, MX5, MX50, MX51, MX52, MX53, MX54, MX57, MX58, MX59, MX6, MX60, MX61, MX62, MX63, MX64, MX65, MX7, MX8, MX9: footprint PCM_marbastlib-mx:SW_MX_HS_CPG151101S11_1u -> marbastlib-mx:SW_MX_HS_CPG151101S11_1u
- MX55: renamed from MX56; footprint PCM_marbastlib-mx:SW_MX_HS_CPG151101S11_1u -> marbastlib-mx:SW_MX_HS_CPG151101S11_1u
- MX56: renamed from MX55; footprint PCM_marbastlib-mx:SW_MX_HS_CPG151101S11_1u -> marbastlib-mx:SW_MX_HS_CPG151101S11_1u
- Q1: value AO3401A -> 2N7002
- R1, R10, R2, R3, R4, R5, R6, R7, R8, R9: footprint (none) -> Resistor_SMD:R_0402_1005Metric
- SW1: footprint (none) -> Button_Switch_SMD:SW_SPDT_CK_JS102011SAQN
- SW2, SW3: value T-1187-A-B-A-B -> TS-1187-A-B-A-B; footprint (none) -> Button_Switch_SMD:SW_Push_1P1T_XKB_TS-1187A
- TP1, TP4: footprint (none) -> TestPoint:TestPoint_Pad_D1.0mm
- U3: footprint PCM_marbastlib-various:nRF52840_holyiot_18010 -> marbastlib-various:nRF52840_holyiot_18010
- U4: value XC6206PxxxMR -> XC6206P332MR-G
Connections:
- net COL10: now also MX62.1; no longer MX63.1
- net COL11: now also MX63.1; no longer MX62.1
- net COL12: no longer MX64.1
- net COL13: now also MX64.1; no longer MX42.1, MX65.1
- net COL14: now also MX42.1, MX65.1
- net ROW1: now also D21.1 (K), D22.1 (K), D23.1 (K), D24.1 (K), D25.1 (K), D26.1 (K), D27.1 (K), D28.1 (K), D29.1 (K), D30.1 (K), D31.1 (K)
Other:
- moved on the sheet: D64, D65, J2, MX62, MX63

Commit message: first final
Parts:
- removed C1, C2: 100nF, Capacitor_SMD:C_0402_1005Metric, symbol Device:C_Small
- removed D1: BSD3C051V, Diode_SMD:D_SOD-323, symbol Device:D_Small
- removed L2: BLM15PX121N1D, Inductor_SMD:L_0402_1005Metric, symbol Device:L_Small
- removed TP1, TP4: TestPoint, TestPoint:TestPoint_Pad_D1.0mm, symbol Connector:TestPoint
- L1: value BLM15PX121N1D -> BLM15PX121SN1D
Connections:
- net GNDPWR is gone; now on net GND: R1.1, R2.2
- net +5V: now also F1.2
- net COL0: now also U3.13 (P0.05-A); no longer U3.11 (P0.31-LF-A)
- net COL1: now also U3.5 (P1.15-LF); no longer U3.10 (P0.30-LF-A)
- net COL11: now also U3.33 (P1.04-LF); no longer U3.29 (P1.01-LF)
- net COL12: now also MX64.1, U3.34 (P1.06-LF); no longer U3.28 (P1.03-LF)
- net COL13: now also U3.35 (P0.09-LF-NFC); no longer MX64.1, U3.27 (P1.00)
- net COL14: now also U3.2 (P1.11-LF); no longer U3.26 (P0.22)
- net COL2: now also U3.6 (P0.03-LF-A); no longer U3.9 (P0.29-LF-A)
- net COL3: now also U3.7 (P0.02-LF-A); no longer U3.8 (P0.28-LF-A)
- net COL4: now also U3.8 (P0.28-LF-A); no longer U3.7 (P0.02-LF-A)
- net COL5: now also U3.26 (P0.22); no longer U3.6 (P0.03-LF-A)
- net COL6: now also U3.27 (P1.00); no longer U3.5 (P1.15-LF)
- net COL7: now also U3.28 (P1.03-LF); no longer U3.4 (P1.13-LF)
- net COL8: now also U3.36 (P0.10-LF-NFC); no longer U3.3 (P1.10-LF)
- net COL9: now also U3.29 (P1.01-LF); no longer U3.2 (P1.11-LF)
- net GND: now also J1.A1_B12 (GND), J1.B1_A12 (GND), J1.S1 (SHIELD), J1.S2 (SHIELD), J1.S3 (SHIELD), J1.S4 (SHIELD)
- net ROW0: now also U3.9 (P0.29-LF-A); no longer U3.15 (P0.07)
- net ROW1: now also U3.12 (P0.04-A); no longer U3.16 (P1.09)
- net ROW2: now also U3.11 (P0.31-LF-A); no longer U3.17 (P0.12)
- net ROW3: now also U3.10 (P0.30-LF-A); no longer U3.18 (P0.23)
- net ROW4: now also U3.3 (P1.10-LF); no longer U3.19 (P0.21)
- no-connect marks 29 -> 24

Commit message: else
Parts:
- C3, C4, C5: footprint Capacitor_SMD:C_0402_1005Metric -> Capacitor_SMD:C_0603_1608Metric
- C6, C7: footprint Capacitor_SMD:C_1812_4532Metric -> Capacitor_SMD:C_1206_3216Metric
- R3: footprint Resistor_SMD:R_0402_1005Metric -> Resistor_SMD:R_0603_1608Metric
Changed lines of the file:
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@@
 			)
 		)
-		(property "Footprint" "Capacitor_SMD:C_0402_1005Metric"
+		(property "Footprint" "Capacitor_SMD:C_0603_1608Metric"
 			(at 156.21 29.21 0)
 			(effects
@@
 			)
 		)
-		(property "Footprint" "Capacitor_SMD:C_1812_4532Metric"
+		(property "Footprint" "Capacitor_SMD:C_1206_3216Metric"
 			(at 241.3 87.63 0)
 			(effects
@@
 			)
 		)
-		(property "Footprint" "Resistor_SMD:R_0402_1005Metric"
+		(property "Footprint" "Resistor_SMD:R_0603_1608Metric"
 			(at 167.64 52.07 0)
 			(effects
@@
 			)
 		)
-		(property "Footprint" "Capacitor_SMD:C_0402_1005Metric"
+		(property "Footprint" "Capacitor_SMD:C_0603_1608Metric"
 			(at 209.55 39.37 0)
 			(effects
@@
 			)
 		)
-		(property "Footprint" "Capacitor_SMD:C_1812_4532Metric"
+		(property "Footprint" "Capacitor_SMD:C_1206_3216Metric"
 			(at 222.25 87.63 0)
 			(effects
@@
 			)
 		)
-		(property "Footprint" "Capacitor_SMD:C_0402_1005Metric"
+		(property "Footprint" "Capacitor_SMD:C_0603_1608Metric"
 			(at 217.17 33.02 0)
 			(effects
