File: obscura60/H360.kicad_sch (KiCad schematic)
At the start: 158 parts, among them J1 TYPE-C-31-M-12, J2 S2B-PH-SM4-TB, Q1 2N7002, SW1 PWR, SW2 TS-1187-A-B-A-B, SW3 TS-1187-A-B-A-B, U1 SRV05-4-P-T7, U3 nRF52840_holyiot_18010, U4 XC6206P332MR-G, U5 BQ24075RGT

Commit message: update
Parts:
- R8: value 10k -> 100k
Changed lines of the file:
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@@
 	)
 	(global_label "SYSOFF"
-		(shape input)
+		(shape output)
 		(at 246.38 33.02 180)
 		(fields_autoplaced yes)
@@
 			)
 		)
-		(property "Value" "10k"
+		(property "Value" "100k"
 			(at 269.24 29.2099 0)
 			(effects
